File: HW/Circuitos electronicos/Circuitos_ISE/Circuito_consumo_sch.kicad_sch (KiCad schematic)
At the start: 16 parts, among them U3 TL074, U77 TL074

Commit message: Esquematicos finales
Parts:
- added U2: TL074, symbol Amplifier_Operational:TL074
- U77: value TL074 -> LM224
Connections:
- net GND_A: now also R83.1
- net Vbat-: now also R84.2, U2.11 (V-)
- net V_Cons renamed PC3
- new net 10V: U2.4 (V+)
Other:
- moved on the sheet: BT3, BT4, R29, R30, R31, R32, R33, R34, R82, R83, R84, R85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
