File: HW/Circuitos electronicos/Circuitos_ISE/Sensores_DIgitales.kicad_sch (KiCad schematic)
At the start: 6 parts, among them U10 PCF8575DBR, U11 PCF8575DBR, U12 PCF8575DBR, U8 VL6180X, U9 PCF8575DBR

Commit message: Esquematicos finales
Parts:
- removed U10, U11, U12, U9: PCF8575DBR, Package_SO:SSOP-24_5.3x8.2mm_P0.65mm, symbol Interface_Expansion:PCF8575DBR
- added U9: CAT24C256, symbol Memory_EEPROM:CAT24C256
Connections:
- net PA15: now reaches RFID1.1 (SDA)
- net PC10: now reaches RFID1.2 (SCK)
- net PC11: now reaches RFID1.3 (MOSI)
- net PC12: now reaches RFID1.4 (MISO)
- net Vbat-: now reaches RFID1.6 (GND)
- net Vbat-: now also U8.12 (GND), U8.3 (GND), U8.4 (GND), U8.6 (GND), U9.1 (A0), U9.2 (A1), U9.3 (A2), U9.4 (GND), U9.7 (WP)
- net 3V3: now reaches RFID1.8 (3,3V)
- net PF1: now reaches U8.10 (SCL)
- net 5v: now reaches U8.11 (AVDD)
- net PF0: now reaches U8.9 (SDA)
- new net PF0_S: U9.6 (SCL)
- new net PF1_S: U9.5 (SDA)
- no-connect marks 0 -> 3
Other:
- moved on the sheet: RFID1, U8
