File: HW/Circuitos electronicos/Circuitos_ISE/alimentacion.kicad_sch (KiCad schematic)
At the start: 10 parts, among them J1 Conn_01x02, U1 TL074, U2 TL074, U3 TL074, U4 LM2596S-ADJ, U5 L7805

Commit message: Esquematicos finales
Parts:
- removed U2: TL074, symbol Amplifier_Operational:TL074
Changed lines of the file:
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@@
-	(wire
-		(pts
-			(xy 59.69 45.72) (xy 59.69 49.53)
-		)
-		(stroke
-			(width 0)
-			(type default)
-		)
-	)
 	(wire
 		(pts
@@
 		(pts
 			(xy 135.89 58.42) (xy 144.78 58.42)
-		)
-		(stroke
-			(width 0)
-			(type default)
-		)
-	)
-	(wire
-		(pts
-			(xy 59.69 64.77) (xy 59.69 68.58)
 		)
 		(stroke
@@
 		)
 	)
-	(label "10V"
-		(at 59.69 45.72 0)
-		(effects
-			(font
-				(size 1.27 1.27)
-			)
-			(justify left bottom)
-		)
-	)
 	(label "Vbat-"
 		(at 95.25 83.82 180)
@@
 	(label "V_Cortex"
 		(at 228.6 57.15 0)
-		(effects
-			(font
-				(size 1.27 1.27)
-			)
-			(justify left bottom)
-		)
-	)
-	(label "Vbat-"
-		(at 59.69 68.58 0)
 		(effects
 			(font
@@
 				)
 			)
-		)
-	)
-	(symbol
-		(lib_id "Amplifier_Operational:TL074")
-		(at 62.23 57.15 0)
-		(unit 5)
-		(exclude_from_sim no)
-		(in_bom yes)
-		(on_board yes)
-		(dnp no)
-		(fields_autoplaced yes)
-		(property "Reference" "U2"
-			(at 60.96 55.8799 0)
-			(effects
-				(font
-					(size 1.27 1.27)
-				)
-				(justify left)
-			)
-		)
-		(property "Value" "TL074"
-			(at 60.96 58.4199 0)
-			(effects
-				(font
-					(size 1.27 1.27)
-				)
-				(justify left)
-			)
-		)
-		(property "Footprint" ""
-			(at 60.96 54.61 0)
-			(effects
-				(font
-					(size 1.27 1.27)
-				)
-				(hide yes)
-			)
-		)
-		(property "Datasheet" "http://www.ti.com/lit/ds/symlink/tl071.pdf"
-			(at 63.5 52.07 0)
-			(effects
-				(font
-					(size 1.27 1.27)
-				)
-				(hide yes)
-			)
-		)
-		(property "Description" "Quad Low-Noise JFET-Input Operational Amplifiers, DIP-14/SOIC-14"
-			(at 62.23 57.15 0)
-			(effects
-				(font
-					(size 1.27 1.27)
-				)
-				(hide yes)
-			)
-		)
-		(pin "10"
-		)
-		(pin "14"
-		)
-		(pin "5"
-		)
-		(pin "4"
-		)
-		(pin "9"
-		)
-		(pin "11"
-		)
-		(pin "6"
-		)
-		(pin "2"
-		)
-		(pin "3"
-		)
-		(pin "1"
-		)
-		(pin "7"
-		)
-		(pin "8"
-		)
-		(pin "12"
-		)
-		(pin "13"
-		)
-		(instances
-			(project "Circuitos_ISE"
-				(path "/fc1c7a48-e258-41da-82b5-172f051ec090/f59b483d-e1b5-4aee-ae4d-c4afa44cd173"
-					(reference "U2")
-					(unit 5)
-				)
-			)
