File: HW/Circuitos electronicos/Circuitos_ISE/filtro_activo.kicad_sch (KiCad schematic)
At the start: 17 parts, among them U1 TL074

Commit message: Esquematicos finales
Parts:
- removed RG4: R_Potentiometer_US, symbol Device:R_Potentiometer_US
- added R36: 100K, symbol Device:R_US
- added U3: TL074, symbol Amplifier_Operational:TL074
Connections:
- net PC0: now also R37.2, R36.1
- net Vbat-: now also U3.11 (V-)
- net Vmic: now also R36.2
- new net 10V: U3.4 (V+)
Changed lines of the file:
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@@
+	)
+	(junction
+		(at 227.33 92.71)
+		(diameter 0)
+		(color 0 0 0 0)
 	)
 	(junction
@@
 	(wire
 		(pts
+			(xy 236.22 90.17) (xy 236.22 92.71)
+		)
+		(stroke
+			(width 0)
+			(type default)
+		)
+	)
+	(wire
+		(pts
 			(xy 160.02 57.15) (xy 170.18 57.15)
 		)
@@
 	(wire
 		(pts
-			(xy 231.14 86.36) (xy 247.65 86.36)
+			(xy 236.22 90.17) (xy 252.73 90.17)
 		)
 		(stroke
@@
 	(wire
 		(pts
-			(xy 227.33 90.17) (xy 227.33 99.06)
+			(xy 227.33 90.17) (xy 227.33 92.71)
 		)
 		(stroke
@@
 	(wire
 		(pts
-			(xy 247.65 86.36) (xy 247.65 85.09)
+			(xy 252.73 90.17) (xy 252.73 88.9)
 		)
 		(stroke
@@
 	(wire
 		(pts
+			(xy 227.33 92.71) (xy 227.33 99.06)
+		)
+		(stroke
+			(width 0)
+			(type default)
+		)
+	)
+	(wire
+		(pts
 			(xy 160.02 67.31) (xy 151.13 67.31)
 		)
@@
 	(wire
 		(pts
+			(xy 237.49 57.15) (xy 237.49 60.96)
+		)
+		(stroke
+			(width 0)
+			(type default)
+		)
+	)
+	(wire
+		(pts
 			(xy 53.34 95.25) (xy 53.34 104.14)
 		)
@@
 	(wire
 		(pts
+			(xy 237.49 39.37) (xy 237.49 41.91)
+		)
+		(stroke
+			(width 0)
+			(type default)
+		)
+	)
+	(wire
+		(pts
 			(xy 109.22 77.47) (xy 120.65 77.47)
 		)
@@
 		(pts
 			(xy 152.4 57.15) (xy 160.02 57.15)
+		)
+		(stroke
+			(width 0)
+			(type default)
+		)
+	)
+	(wire
+		(pts
+			(xy 227.33 92.71) (xy 236.22 92.71)
 		)
 		(stroke
@@
 		)
 	)
+	(label "Vbat-"
+		(at 237.49 60.96 0)
+		(effects
+			(font
+				(size 1.27 1.27)
+			)
+			(justify left bottom)
+		)
+	)
+	(label "10V"
+		(at 237.49 39.37 180)
+		(effects
+			(font
+				(size 1.27 1.27)
+			)
+			(justify right bottom)
+		)
+	)
 	(label "Vmic"
 		(at 210.82 80.01 0)
@@
 	)
 	(label "PC0"
-		(at 247.65 85.09 0)
+		(at 252.73 88.9 0)
 		(effects
 			(font
@@
 				(path "/fc1c7a48-e258-41da-82b5-172f051ec090/3a0694a3-df0f-4d25-944d-88c4e1913a02"
 					(reference "R37")
+					(unit 1)
+				)
+			)
+		)
+	)
+	(symbol
+		(lib_id "Device:R_US")
+		(at 227.33 86.36 180)
+		(unit 1)
+		(exclude_from_sim no)
+		(in_bom yes)
+		(on_board yes)
+		(dnp no)
+		(property "Reference" "R36"
+			(at 220.98 86.36 90)
+			(effects
+				(font
+					(size 1.27 1.27)
+				)
+			)
+		)
+		(property "Value" "100K"
+			(at 223.52 86.36 90)
+			(effects
+				(font
+					(size 1.27 1.27)
+				)
+			)
+		)
+		(property "Footprint" ""
+			(at 226.314 86.106 90)
+			(effects
+				(font
+					(size 1.27 1.27)
+				)
+				(hide yes)
+			)
+		)
+		(property "Datasheet" "~"
+			(at 227.33 86.36 0)
+			(effects
+				(font
+					(size 1.27 1.27)
+				)
+				(hide yes)
+			)
+		)
+		(property "Description" "Resistor, US symbol"
+			(at 227.33 86.36 0)
+			(effects
+				(font
+					(size 1.27 1.27)
+				)
+				(hide yes)
+			)
+		)
+		(pin "2"
+		)
+		(pin "1"
+		)
+		(instances
+			(project "Circuitos_ISE"
+				(path "/fc1c7a48-e258-41da-82b5-172f051ec090/3a0694a3-df0f-4d25-944d-88c4e1913a02"
+					(reference "R36")
 					(unit 1)
 				)
@@
 				(path "/fc1c7a48-e258-41da-82b5-172f051ec090/3a0694a3-df0f-4d25-944d-88c4e1913a02"
 					(reference "D1")
-					(unit 1)
-				)
-			)
-		)
-	)
-	(symbol
-		(lib_id "Device:R_Potentiometer_US")
-		(at 227.33 86.36 0)
-		(mirror x)
-		(unit 1)
-		(exclude_from_sim no)
-		(in_bom yes)
-		(on_board yes)
-		(dnp no)
-		(property "Reference" "RG4"
-			(at 224.79 85.0899 0)
-			(effects
-				(font
-					(size 1.27 1.27)
-				)
-				(justify right)
-			)
-		)
-		(property "Value" "R_Potentiometer_US"
-			(at 231.394 79.756 0)
-			(effects
-				(font
-					(size 1.27 1.27)
-				)
-				(justify right)
-				(hide yes)
-			)
-		)
-		(property "Footprint" ""
-			(at 227.33 86.36 0)
-			(effects
-				(font
-					(size 1.27 1.27)
-				)
-				(hide yes)
-			)
-		)
-		(property "Datasheet" "~"
-			(at 227.33 86.36 0)
-			(effects
-				(font
-					(size 1.27 1.27)
-				)
-				(hide yes)
-			)
-		)
-		(property "Description" "Potentiometer, US symbol"
-			(at 227.33 86.36 0)
-			(effects
-				(font
-					(size 1.27 1.27)
-				)
-				(hide yes)
-			)
-		)
-		(pin "2"
-		)
-		(pin "3"
-		)
-		(pin "1"
-		)
-		(instances
-			(project "Circuitos_ISE"
-				(path "/fc1c7a48-e258-41da-82b5-172f051ec090/3a0694a3-df0f-4d25-944d-88c4e1913a02"
-					(reference "RG4")
 					(unit 1)
 				)
@@
 				)
 			)
+		)
+	)
+	(symbol
+		(lib_id "Amplifier_Operational:TL074")
+		(at 240.03 49.53 0)
+		(unit 5)
+		(exclude_from_sim no)
+		(in_bom yes)
+		(on_board yes)
+		(dnp no)
+		(fields_autoplaced yes)
+		(property "Reference" "U3"
+			(at 238.76 48.2599 0)
+			(effects
+				(font
+					(size 1.27 1.27)
+				)
+				(justify left)
+			)
+		)
+		(property "Value" "TL074"
+			(at 238.76 50.7999 0)
+			(effects
+				(font
+					(size 1.27 1.27)
+				)
+				(justify left)
+			)
+		)
+		(property "Footprint" ""
+			(at 238.76 46.99 0)
+			(effects
+				(font
+					(size 1.27 1.27)
+				)
+				(hide yes)
+			)
+		)
+		(property "Datasheet" "http://www.ti.com/lit/ds/symlink/tl071.pdf"
+			(at 241.3 44.45 0)
+			(effects
+				(font
+					(size 1.27 1.27)
+				)
+				(hide yes)
+			)
+		)
+		(property "Description" "Quad Low-Noise JFET-Input Operational Amplifiers, DIP-14/SOIC-14"
+			(at 240.03 49.53 0)
+			(effects
+				(font
+					(size 1.27 1.27)
+				)
+				(hide yes)
+			)
+		)
+		(pin "11"
+		)
+		(pin "12"
+		)
+		(pin "6"
+		)
+		(pin "10"
+		)
+		(pin "5"
+		)
+		(pin "13"
+		)
+		(pin "14"
+		)
+		(pin "8"
+		)
+		(pin "9"
+		)
+		(pin "1"
+		)
+		(pin "4"
+		)
+		(pin "2"
+		)
+		(pin "7"
+		)
+		(pin "3"
+		)
+		(instances
+			(project "Circuitos_ISE"
+				(path "/fc1c7a48-e258-41da-82b5-172f051ec090/3a0694a3-df0f-4d25-944d-88c4e1913a02"
+					(reference "U3")
+					(unit 5)
+				)
+			)
